Commit message: initialize

File: Assets/armstrong_description/armstrong.urdf.xacro (robot description, xacro)
@@ -438,5 +438,5 @@
         <child  link="link_1"/>
         <origin rpy="0 0 0" xyz="0 0.15508 0.076053"/>
-        <axis xyz="0 0 1"/>
+        <axis xyz="0 -1 0"/>
         <limit lower="-1.5708" upper="1.5708" effort="24" velocity="6.07"/>
     </joint>
@@ -493,5 +493,5 @@
         <origin rpy="0 0 0" xyz="0.01853 -0.000527 0.05403"/>
         <axis xyz="0 1 0"/>
-        <limit lower="-0.40" upper="0" effort="10" velocity="6.07"/>
+        <limit lower="-100" upper="100" effort="10" velocity="6.07"/>
     </joint>
    <xacro:transmission_block joint_name="joint_r_finger"/>
@@ -502,5 +502,5 @@
         <origin rpy="0 0 0" xyz="-0.01853 -0.000527 0.05403"/>
         <axis xyz="0 1 0"/>
-        <limit lower="0" upper="0.40" effort="10" velocity="6.07"/>
+        <limit lower="-100" upper="100" effort="10" velocity="6.07"/>
     </joint>
    <xacro:transmission_block joint_name="joint_l_finger"/>
